File: KiCAD/xirtam.sch (KiCad schematic (older format))
At the start: 25 parts, among them J1 Exp Header, J2 Matrix, J3 Power, J4 JTAG, J5 Bootloader, P1 USB_A, SW1 SW_Push_SPDT, U1 MT093APR1, U2 AT90USB1287, Y1 16 MHz Crystal

Commit message: Add in-line connector layout to PCB, no routing
Parts:
- removed J1: Exp Header, Connector_PinHeader_2.54mm:PinHeader_1x10_P2.54mm_Horizontal, symbol xirtam-rescue:CONN_01X10
- removed J2: Matrix, Connector_PinHeader_2.54mm:PinHeader_1x20_P2.54mm_Horizontal, symbol Connector:Conn_01x20_Male
- added J1: Conn_01x15_Female, Connector_PinSocket_2.54mm:PinSocket_1x15_P2.54mm_Horizontal, symbol Connector:Conn_01x15_Female
- added J2: Conn_01x15_Male, Connector_PinHeader_2.54mm:PinHeader_1x15_P2.54mm_Horizontal, symbol Connector:Conn_01x15_Male
Connections:
- wire segments 172 -> 182
- no-connect marks 28 -> 40
Other:
- note added: "1Y0"
- note added: "1Y1"
- note added: "2Y0"
- note added: "2Y1"
- note added: "2Y2"
- note added: "2Y3"
- note added: "INT10"
- note added: "INT3"
- note added: "INT4"
- note added: "INT5"
- note added: "INT6"
- note added: "INT7"
- note added: "INT8"
- note added: "INT9"
- note added: "P5"
Changed lines of the file:
@@
 encoding utf-8
 Sheet 1 1
-Title "xirtam"
+Title "xirtam TI-99/4A"
 Date "2017-02-16"
 Rev "2.0"
@@
 NoConn ~ 5800 2600
 NoConn ~ 5800 2700
-Wire Wire Line
-	5800 4700 6100 4700
-Wire Wire Line
-	5800 4800 6100 4800
-Wire Wire Line
-	5800 4900 6100 4900
-Wire Wire Line
-	5800 5000 6100 5000
-Wire Wire Line
-	5800 5100 6100 5100
-Wire Wire Line
-	5800 5200 6100 5200
-Wire Wire Line
-	5800 5300 6100 5300
-Wire Wire Line
-	5800 5400 6100 5400
-$Comp
-L power:+5V #PWR013
-U 1 1 590F1572
-P 6700 5550
-F 0 "#PWR013" H 6700 5400 50  0001 C CNN
-F 1 "+5V" H 6700 5690 50  0000 C CNN
-F 2 "" H 6700 5550 50  0000 C CNN
-F 3 "" H 6700 5550 50  0000 C CNN
-	1    6700 5550
-	1    0    0    -1
-$EndComp
-Wire Wire Line
-	6100 5600 6050 5600
-Wire Wire Line
-	6100 5500 5950 5500
-Wire Wire Line
-	5950 5500 5950 5800
-Connection ~ 4600 5800
 NoConn ~ 5800 3100
 NoConn ~ 5800 3200
@@
 	2950 3400 3100 3400
 Wire Wire Line
-	4600 5800 5950 5800
-Wire Wire Line
 	4500 6950 4800 6950
 Wire Wire Line
@@
 Wire Wire Line
 	5800 4500 7400 4500
-Wire Wire Line
-	6050 5600 6050 5800
-Wire Wire Line
-	6050 5800 6700 5800
-Wire Wire Line
-	6700 5800 6700 5550
 Wire Wire Line
 	5800 2900 6750 2900
@@
 Wire Wire Line
 	8100 4750 8100 4950
-$Comp
-L Connector:Conn_01x20_Male J2
-U 1 1 60989A86
-P 9850 3600
-F 0 "J2" H 9822 3574 50  0000 R CNN
-F 1 "Matrix" H 9822 3483 50  0000 R CNN
-F 2 "Connector_PinHeader_2.54mm:PinHeader_1x20_P2.54mm_Horizontal" H 9850 3600 50  0001 C CNN
-F 3 "~" H 9850 3600 50  0001 C CNN
-	1    9850 3600
-	-1   0    0    1
-$EndComp
-Wire Wire Line
-	8800 2600 9650 2600
-Wire Wire Line
-	9650 2700 8800 2700
-Wire Wire Line
-	8800 2800 9650 2800
-Wire Wire Line
-	9650 2900 8800 2900
-Wire Wire Line
-	8800 3000 9650 3000
-Wire Wire Line
-	9650 3100 8800 3100
-Wire Wire Line
-	8800 3200 9650 3200
-Wire Wire Line
-	9650 3300 8800 3300
-Wire Wire Line
-	8800 3400 9650 3400
-Wire Wire Line
-	9650 3500 8800 3500
-Wire Wire Line
-	8800 3600 9650 3600
-Wire Wire Line
-	9650 3700 8800 3700
-Wire Wire Line
-	8800 3800 9650 3800
-Wire Wire Line
-	9650 3900 8800 3900
-Wire Wire Line
-	8800 4000 9650 4000
-Wire Wire Line
-	9650 4100 8800 4100
-Wire Wire Line
-	8800 4200 9650 4200
-Wire Wire Line
-	9650 4300 8800 4300
-Wire Wire Line
-	8800 4400 9650 4400
-Wire Wire Line
-	9650 4500 8800 4500
 Text GLabel 6400 1100 0    60   Input ~ 0
 TCK
@@
 NoConn ~ 5800 2100
 NoConn ~ 5800 2000
-NoConn ~ 5200 5100
-$Comp
-L xirtam-rescue:CONN_01X10 J1
-U 1 1 590F0D71
-P 6300 5150
-F 0 "J1" H 6300 5700 50  0000 C CNN
-F 1 "Exp Header" V 6400 5150 50  0000 C CNN
-F 2 "Connector_PinHeader_2.54mm:PinHeader_1x10_P2.54mm_Horizontal" H 6300 5150 50  0001 C CNN
-F 3 "" H 6300 5150 50  0001 C CNN
-	1    6300 5150
-	1    0    0    1
-$EndComp
+$Comp
+L Connector:Conn_01x15_Female J1
+U 1 1 60DE32D9
+P 10000 5050
+F 0 "J1" V 10073 5030 50  0000 C CNN
+F 1 "Conn_01x15_Female" V 10164 5030 50  0000 C CNN
+F 2 "Connector_PinSocket_2.54mm:PinSocket_1x15_P2.54mm_Horizontal" H 10000 5050 50  0001 C CNN
+F 3 "~" H 10000 5050 50  0001 C CNN
+	1    10000 5050
+	0    1    1    0
+$EndComp
+NoConn ~ 5800 4700
+NoConn ~ 5800 4800
+NoConn ~ 5800 4900
+NoConn ~ 5800 5000
+NoConn ~ 5800 5100
+NoConn ~ 5800 5200
+NoConn ~ 5800 5300
+NoConn ~ 5800 5400
+Text Notes 10700 2300 1    60   ~ 0
+INT5
+Text Notes 10600 2300 1    60   ~ 0
+INT6
+Text Notes 10500 2300 1    60   ~ 0
+INT8
+Text Notes 10400 2300 1    60   ~ 0
+INT4
+Text Notes 10300 2300 1    60   ~ 0
+INT3
+Text Notes 10200 2300 1    60   ~ 0
+P5
+Text Notes 10100 2300 1    60   ~ 0
+INT7
+Text Notes 10000 2300 1    60   ~ 0
+1Y1
+Text Notes 9900 2300 1    60   ~ 0
+1Y0
+Text Notes 9800 2300 1    60   ~ 0
+INT9
+Text Notes 9700 2300 1    60   ~ 0
+INT10
+Text Notes 9600 2300 1    60   ~ 0
+2Y0
+Text Notes 9500 2300 1    60   ~ 0
+2Y1
+Text Notes 9400 2300 1    60   ~ 0
+2Y2
+Text Notes 9300 2300 1    60   ~ 0
+2Y3
+$Comp
+L Connector:Conn_01x15_Male J2
+U 1 1 60EDF4D7
+P 10000 1900
+F 0 "J2" V 9835 1878 50  0000 C CNN
+F 1 "Conn_01x15_Male" V 9926 1878 50  0000 C CNN
+F 2 "Connector_PinHeader_2.54mm:PinHeader_1x15_P2.54mm_Horizontal" H 10000 1900 50  0001 C CNN
+F 3 "~" H 10000 1900 50  0001 C CNN
+	1    10000 1900
+	0    1    1    0
+$EndComp
+Wire Wire Line
+	10100 2100 10100 2600
+Wire Wire Line
+	10600 2100 10600 3300
+Wire Wire Line
+	10200 2100 10200 4000
+Wire Wire Line
+	9600 2100 9600 3700
+Wire Wire Line
+	9500 2100 9500 3600
+Wire Wire Line
+	9400 2100 9400 3500
+Wire Wire Line
+	10300 2100 10300 3000
+Wire Wire Line
+	9800 2100 9800 2700
+Wire Wire Line
+	9700 2100 9700 2800
+Wire Wire Line
+	10700 2100 10700 2900
+Wire Wire Line
+	10400 2100 10400 3100
+Wire Wire Line
+	10500 2100 10500 3200
+Wire Wire Line
+	10000 2100 10000 3900
+Wire Wire Line
+	9900 2100 9900 3800
+Wire Wire Line
+	9300 2100 9300 3400
+Wire Wire Line
+	8800 2900 10700 2900
+Connection ~ 10700 2900
+Wire Wire Line
+	10700 2900 10700 4850
+Wire Wire Line
+	8800 3300 10600 3300
+Connection ~ 10600 3300
+Wire Wire Line
+	10600 3300 10600 4850
+Wire Wire Line
+	8800 3200 10500 3200
+Connection ~ 10500 3200
+Wire Wire Line
+	10500 3200 10500 4850
+Wire Wire Line
+	8800 3100 10400 3100
+Connection ~ 10400 3100
+Wire Wire Line
+	10400 3100 10400 4850
+Wire Wire Line
+	8800 3000 10300 3000
+Connection ~ 10300 3000
+Wire Wire Line
+	10300 3000 10300 4850
+Wire Wire Line
+	8800 2600 10100 2600
+Connection ~ 10100 2600
+Wire Wire Line
+	10100 2600 10100 4850
+Wire Wire Line
+	8800 2700 9800 2700
+Connection ~ 9800 2700
+Wire Wire Line
+	9800 2700 9800 4850
+Wire Wire Line
+	8800 2800 9700 2800
+Connection ~ 9700 2800
+Wire Wire Line
+	9700 2800 9700 4850
+Wire Wire Line
+	8800 4000 10200 4000
+Connection ~ 10200 4000
+Wire Wire Line
+	10200 4000 10200 4850
+Wire Wire Line
+	8800 3900 10000 3900
+Connection ~ 10000 3900
+Wire Wire Line
+	10000 3900 10000 4850
+Wire Wire Line
+	8800 3800 9900 3800
+Connection ~ 9900 3800
+Wire Wire Line
+	9900 3800 9900 4850
+Wire Wire Line
+	8800 3700 9600 3700
+Connection ~ 9600 3700
+Wire Wire Line
+	9600 3700 9600 4850
+Wire Wire Line
+	8800 3600 9500 3600
+Connection ~ 9500 3600
+Wire Wire Line
+	9500 3600 9500 4850
+Wire Wire Line
+	8800 3500 9400 3500
+Connection ~ 9400 3500
+Wire Wire Line
+	9400 3500 9400 4850
+Wire Wire Line
+	8800 3400 9300 3400
+Connection ~ 9300 3400
+Wire Wire Line
+	9300 3400 9300 4850
+NoConn ~ 8800 4100
+NoConn ~ 8800 4200
+NoConn ~ 8800 4300
+NoConn ~ 8800 4400
+NoConn ~ 8800 4500
 $EndSCHEMATC

Commit message: Add serial port, fix bugs, make SmallyMouse2 compatible
Parts:
- added J6: Debug Serial Port, symbol Connector:Conn_01x04_Male
- J1: value Conn_01x15_Female -> To Computer
- J2: value Conn_01x15_Male -> To Keyboard
- SW1: value SW_Push_SPDT -> Reset
- Y1: value 16 MHz Crystal -> 16 MHz
Connections:
- net +5V: now also J6.4 (Pin_4)
- net GND: now also J6.1 (Pin_1)
- net ~RESET: now also SW1.3 (C); no longer SW1.1 (A)
- net at U2.10 ((SS/PCINT0)PB0): no longer U1.3 (RESET)
- net at U2.11 ((PCINT1/SCLK)PB1): no longer U1.20 (STROBE)
- net at U2.25 ((OC0B/SCL/INT0)PD0): now also U1.20 (STROBE)
- net at U2.26 ((OC2B/SDA/INT1)PD1): now also U1.42 (DATA)
- net RxD: now reaches U2.27 ((RXD1/INT2)PD2)
- net RxD: now also J6.3 (Pin_3)
- net TxD: now reaches U2.28 ((TXD1/INT3)PD3)
- net TxD: now also J6.2 (Pin_2)
- net at U2.29 ((ICP1)PD4): now also U1.3 (RESET)
- net at U2.35 ((A8)PC0): now also U1.5 (AX0)
- net at U2.36 ((A9)PC1): now also U1.24 (AX1); no longer U1.5 (AX0)
- net at U2.37 ((A10)PC2): now also U1.25 (AX2); no longer U1.24 (AX1)
- net at U2.38 ((A11/T.3)PC3): now also U1.4 (AX3); no longer U1.25 (AX2)
- net at U2.39 ((A12/OC.3C)PC4): now also U1.26 (AY0); no longer U1.4 (AX3)
- net at U2.40 ((A13/OC.3B)PC5): now also U1.27 (AY1); no longer U1.26 (AY0)
- net at U2.41 ((A14/OC.3A)PC6): now also U1.2 (AY2); no longer U1.27 (AY1)
- net at U2.42 ((A15/IC.3/CLKO)PC7): no longer U1.2 (AY2)
- no-connect marks 40 -> 38
Other:
- moved on the sheet: J1, J2, R2, U1

Commit message: New PCB layout
Parts:
- removed C7, C8, C9: 100nF, Capacitor_SMD:C_0603_1608Metric_Pad1.05x0.95mm_HandSolder, symbol Device:C
- removed J1: To Computer, Connector_PinSocket_2.54mm:PinSocket_1x15_P2.54mm_Horizontal, symbol Connector:Conn_01x15_Female
- removed J2: To Keyboard, Connector_PinHeader_2.54mm:PinHeader_1x15_P2.54mm_Horizontal, symbol Connector:Conn_01x15_Male
- removed SW1: Reset, Button_Switch_SMD:SW_Push_1P1T_NO_6x6mm_H9.5mm, symbol Switch:SW_Push_SPDT
- added J1: Conn_01x28_Male, Connector_PinHeader_2.54mm:PinHeader_1x28_P2.54mm_Horizontal, symbol Connector:Conn_01x28_Male
- added J2: Conn_01x28_Female, Connector_PinSocket_2.54mm:PinSocket_1x28_P2.54mm_Horizontal, symbol Connector:Conn_01x28_Female
- added M1: MatrixInterconnectMatrix, Jumper:matrixinterconnectmatrix, symbol Jumper:MatrixInterconnectMatrix
- added SW1: Reset, Button_Switch_SMD:SW_SPST_FSMSM, symbol Switch:SW_SPST
- J6: footprint (none) -> Connector_PinHeader_2.54mm:PinHeader_1x04_P2.54mm_Horizontal
- renumbered C10 to C7, C11 to C8
Connections:
- net +5V: now also M1.27 (Y27)
- net GND: now also M1.28 (Y28), SW1.1 (A)
- net ~RESET: now also SW1.2 (B)
- net at U1.1 (Y3): now also M1.4 (Y4)
- net at U1.10 (X7): now also M1.16 (Y16)
- net at U1.11 (X8): now also M1.17 (Y17)
- net at U1.12 (X9): now also M1.18 (Y18)
- net at U1.13 (X10): now also M1.19 (Y19)
- net at U1.14 (X11): now also M1.20 (Y20)
- net at U1.18 (Y7): now also M1.8 (Y8)
- net at U1.19 (Y6): now also M1.7 (Y7)
- net at U1.21 (Y5): now also M1.6 (Y6)
- net at U1.23 (Y4): now also M1.5 (Y5)
- net at U1.32 (X5): now also M1.14 (Y14)
- net at U1.33 (X4): now also M1.13 (Y13)
- net at U1.34 (X3): now also M1.12 (Y12)
- net at U1.35 (X2): now also M1.11 (Y11)
- net at U1.36 (X1): now also M1.10 (Y10)
- net at U1.37 (X0): now also M1.9 (Y9)
- net at U1.40 (Y0): now also M1.1 (Y1)
- net at U1.41 (Y1): now also M1.2 (Y2)
- net at U1.43 (Y2): now also M1.3 (Y3)
- net at U1.9 (X6): now also M1.15 (Y15)
- new net: J1.1 (Pin_1), M1.29 (XA1)
- new net: J1.2 (Pin_2), M1.30 (XA2)
- new net: J1.3 (Pin_3), M1.31 (XA3)
- new net: J1.4 (Pin_4), M1.32 (XA4)
- new net: J1.5 (Pin_5), M1.33 (XA5)
- new net: J1.6 (Pin_6), M1.34 (XA6)
- new net: J1.7 (Pin_7), M1.35 (XA7)
- new net: J1.8 (Pin_8), M1.36 (XA8)
- new net: J1.9 (Pin_9), M1.37 (XA9)
- new net: J1.10 (Pin_10), M1.38 (XA10)
- new net: J1.11 (Pin_11), M1.39 (XA11)
- new net: J1.12 (Pin_12), M1.40 (XA12)
- new net: J1.13 (Pin_13), M1.41 (XA13)
- new net: J1.14 (Pin_14), M1.42 (XA14)
- new net: J1.15 (Pin_15), M1.43 (XA15)
- new net: J1.16 (Pin_16), M1.44 (XA16)
- new net: J1.17 (Pin_17), M1.45 (XA17)
- new net: J1.18 (Pin_18), M1.46 (XA18)
- new net: J1.19 (Pin_19), M1.47 (XA19)
- new net: J1.20 (Pin_20), M1.48 (XA20)
- new net: J1.21 (Pin_21), M1.49 (XA21)
- new net: J1.22 (Pin_22), M1.50 (XA22)
- new net: J1.23 (Pin_23), M1.51 (XA23)
- new net: J1.24 (Pin_24), M1.52 (XA24)
- new net: J1.25 (Pin_25), M1.53 (XA25)
- new net: J1.26 (Pin_26), M1.54 (XA26)
- new net: J1.27 (Pin_27), M1.55 (XA27)
- new net: J1.28 (Pin_28), M1.56 (XA28)
- new net: J2.1 (Pin_1), M1.57 (XB1)
- new net: J2.2 (Pin_2), M1.58 (XB2)
- new net: J2.3 (Pin_3), M1.59 (XB3)
- new net: J2.4 (Pin_4), M1.60 (XB4)
- new net: J2.5 (Pin_5), M1.61 (XB5)
- new net: J2.6 (Pin_6), M1.62 (XB6)
- new net: J2.7 (Pin_7), M1.63 (XB7)
- new net: J2.8 (Pin_8), M1.64 (XB8)
- new net: J2.9 (Pin_9), M1.65 (XB9)
- new net: J2.10 (Pin_10), M1.66 (XB10)
- new net: J2.11 (Pin_11), M1.67 (XB11)
- new net: J2.12 (Pin_12), M1.68 (XB12)
- new net: J2.13 (Pin_13), M1.69 (XB13)
- new net: J2.14 (Pin_14), M1.70 (XB14)
- new net: J2.15 (Pin_15), M1.71 (XB15)
- new net: J2.16 (Pin_16), M1.72 (XB16)
- new net: J2.17 (Pin_17), M1.73 (XB17)
- new net: J2.18 (Pin_18), M1.74 (XB18)
- new net: J2.19 (Pin_19), M1.75 (XB19)
- new net: J2.20 (Pin_20), M1.76 (XB20)
- new net: J2.21 (Pin_21), M1.77 (XB21)
- new net: J2.22 (Pin_22), M1.78 (XB22)
- new net: J2.23 (Pin_23), M1.79 (XB23)
- new net: J2.24 (Pin_24), M1.80 (XB24)
- new net: J2.25 (Pin_25), M1.81 (XB25)
- new net: J2.26 (Pin_26), M1.82 (XB26)
- new net: J2.27 (Pin_27), M1.83 (XB27)
- new net: J2.28 (Pin_28), M1.84 (XB28)
Other:
- note removed: "1Y0"
- note removed: "1Y1"
- note removed: "2Y0"
- note removed: "2Y1"
- note removed: "2Y2"
- note removed: "2Y3"
- note removed: "AT90 Decoupling"
- note removed: "Header Decoupling"
- note removed: "INT10"
- note removed: "INT3"
- note removed: "INT4"
- note removed: "INT5"
- note removed: "INT6"
- note removed: "INT7"
- note removed: "INT8"
- note removed: "INT9"
- note removed: "MT093 Decoupling"
- note removed: "P5"
- moved on the sheet: C5, C6, C7, C8, J3, J4

Commit message: New layout, updated schematic
Parts:
- added U3: 4066, Package_SO:SO-14_5.3x10.2mm_P1.27mm, symbol 4xxx:4066
- J6: value Debug Serial Port -> Debug
Connections:
- net +5V: now also U3.14 (VDD)
- net GND: now also U3.7 (VSS)
- net AUX1: now reaches U2.10 ((SS/PCINT0)PB0)
- net AUX1: now also U3.13
- net AUX2: now reaches U2.11 ((PCINT1/SCLK)PB1)
- net AUX2: now also U3.6
- net AUX3: now reaches U2.12 ((PDI/PCINT2/MOSI)PB2)
- net AUX3: now also U3.12
- net AUX4: now reaches U2.13 ((PDO/PCINT3/MISO)PB3)
- net AUX4: now also U3.5
- net at M1.21 (Y21): now also U3.2
- net at M1.22 (Y22): now also U3.1
- net at M1.23 (Y23): now also U3.9
- net at M1.24 (Y24): now also U3.10
- net at M1.25 (Y25): now also U3.3
- net at M1.26 (Y26): now also U3.11, U3.4, U3.8
- no-connect marks 38 -> 28
Other:
- moved on the sheet: C1, C2, C3, C4, C5, C6, C7, C8, J1, J2, J3, J4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
